Commit message: additions on 20230122

File: src/ackermann_vehicle/urdf/cub_cadet_urdf_joints.xacro (robot description, xacro)
@@ -1,3 +1,4 @@
 <?xml version="1.0"?>
+  <!-- cub_cadet_urdf_joints.xacro -->
 <robot xmlns:xacro="http://www.ros.org/wiki/xacro" >
     <xacro:include filename="inertial_macros.xacro"/>

File: src/ackermann_vehicle/urdf/cub_cadet_urdf_params.xacro (robot description, xacro)
@@ -1,12 +1,12 @@
 <?xml version="1.0"?>
 <robot xmlns:xacro="http://www.ros.org/wiki/xacro" >
-<!-- Wheel and frame Properties for Al's Cub Cadet -->
+<!-- cub_cadet_urdf_params.xacro - Wheel and frame Properties for Al's Cub Cadet -->
   <xacro:property name="hub_dia" value="0.15"/>
 <!-- chassis_length is measured along the x axis, chassis_width
        along the y axis, and chassis_height along the z axis. -->
-  <xacro:property name="chassis_length" value="0.75"/> <!-- 0.505 -->
-  <xacro:property name="chassis_width" value="0.33"/> <!-- 0.25 -->
-  <xacro:property name="chassis_height" value="0.01"/>
-  <xacro:property name="chassis_mass" value="2.788"/>
+  <xacro:property name="chassis_length" value="1.47"/> <!-- wheelbase is 1.27, overall length is 1.47-->
+  <xacro:property name="chassis_width" value="0.97"/> <!-- 0.25 -->
+  <xacro:property name="chassis_height" value="0.81"/>
+  <xacro:property name="chassis_mass" value="150"/>  <!-- my assumption is the value should be in kg-->
   <xacro:property name="main_link" value="base_link" />
   <!-- hub_dia and tire_dia are the diameters of the hub and tire,
@@ -17,7 +17,7 @@
   <xacro:property name="tire_rear_width" value="0.229"/>
   <!-- Wheel spacing is cener to center -->
-  <xacro:property name="wheel_spacing_front" value="0.851"/>
+  <xacro:property name="wheel_spacing_front" value="0.851"/>  <!-- my assumption is the value should be distance between the centerline of each wheel -->
   <xacro:property name="wheel_spacing_rear" value="0.737"/>
-  <xacro:property name="wheelbase" value="1.219"/>
+  <xacro:property name="wheelbase" value="1.27"/>
   <xacro:property name="wheel_mass" value="0.29"/> <!-- ?????? -->
   <xacro:property name="axle_length" value="0.03"/> <!-- 0.05 -->

File: src/ackermann_vehicle/urdf/cub_cadet_urdf_sensors.xacro (robot description, xacro)
@@ -1,9 +1,10 @@
 <?xml version="1.0"?>
 <robot xmlns:xacro="http://www.ros.org/wiki/xacro" >
+<!-- cub_cadet_urdf_sensors.xacro -->
 <!-- ========================= Sensors ========================= -->
   <!-- Fake gps sensor -->
   <joint name="gps0_joint" type="fixed">
     <axis xyz="1 0 0"/> <!-- 0 1 0 -->
-    <origin xyz="0 0 0.53"/>
+    <origin xyz="0.3 -0.1 0.368" rpy= "0 0 0"/>  <!-- copied from vehicle_dimensions_helper.ods -->
     <parent link="base_link"/>
     <child link="gps0_link"/>
@@ -45,57 +46,8 @@
         <velocityGaussianNoise>0.1 0.1 0.1</velocityGaussianNoise>
         <!-- Set the initial GPS location -->
-        <referenceLatitude>45.0122488</referenceLatitude>
-        <referenceLongitude>-93.2439029</referenceLongitude>
+        <referenceLatitude>30.175292</referenceLatitude>
+        <referenceLongitude>-96.512564</referenceLongitude>
     </plugin>
   </gazebo>
-  <!-- Another mock fake gps sensor -->
-  <joint name="gps1_joint" type="fixed">
-    <axis xyz="1 0 0"/> <!-- 0 1 0 -->
-    <origin xyz="0.69 0 0.4575"/>
-    <parent link="base_link"/>
-    <child link="gps1_link"/>
-  </joint>
-  <link name="gps1_link">
-    <inertial>
-      <mass value="0.001"/>
-      <origin rpy="0 0 0" xyz="0 0 0"/>
-      <inertia ixx="0.0001" ixy="0" ixz="0" iyy="0.000001" iyz="0" izz="0.0001"/>
-    </inertial>
-    <visual>
-      <origin rpy="0 0 0" xyz="0 0 0"/>
-      <geometry>
-        <cylinder radius="0.075" length="0.05"/>
-      </geometry>
-      <material name="white"/>
-    </visual>
-    <collision>
-      <origin rpy="0 0 0" xyz="0 0 0"/>
-      <geometry>
-        <cylinder radius="0.075" length="0.04"/>
-      </geometry>
-    </collision>
-  </link>
-  <gazebo reference="gps1_link">
-    <material>Gazebo/White</material>
-  </gazebo>
-<!--
-  <gazebo>
-    <plugin name="my_gps1_sim" filename="libhector_gazebo_ros_gps.so">
-      <alwaysOn>1</alwaysOn>
-      <updateRate>10.0</updateRate>
-      <bodyName>gps1_link</bodyName>
-        <frameId>gps1_link</frameId>
-        <topicName>gps1/fix</topicName>
-        <velocityTopicName>gps1/fix_velocity</velocityTopicName>
-        <drift>0.1 0.1 0.1</drift>
-        <gaussianNoise>0.04 0.04 0.1</gaussianNoise>
-        <velocityDrift>0 0 0</velocityDrift>
-        <velocityGaussianNoise>0.1 0.1 0.1</velocityGaussianNoise>
-   Set the initial GPS location
-        <referenceLatitude>45.0122488</referenceLatitude>
-        <referenceLongitude>-93.2439029</referenceLongitude>
-    </plugin>
-  </gazebo>
--->
   <!-- SickLMS200 Laser Scanner -->
   <joint name="lms200_joint" type="fixed">
@@ -167,5 +119,5 @@
   <joint name="imu_joint" type="fixed">
     <axis xyz="1 0 0"/> <!-- 0 1 0 -->
-    <origin xyz="0.47 -0.08 0.4375 "/>
+    <origin xyz="0.2 0.1 0.216" rpy= "0 0 0"/>  <!-- copied from vehicle_dimensions_helper.ods -->
     <parent link="base_link"/>
     <child link="imu_link"/>
